File: Hardware/Top/D2D-TOP.brd (EAGLE design)
At the start: 38 x 38 mm, 68 parts, among them SW1 SWITCH.MOM, SW2 SWITCH.MOM, U2 NRF52832_MODULE_MDBT42, U4 FT231XS, U5 PCF8523, U6 PHOTOTRANSISTOR

Commit message: push onto repo
Parts:
- removed C2, C5, C6: 1u, LinnesLab-Passives:C0603
- removed C20, C21: 4.7u, LinnesLab-Passives:C0603
- removed CHRG: MCP73831, LinnesLab-Power:SOT23-5
- removed LDO2: MIC5504, LinnesLab-Power:SOT23-5
- removed R11: (no value), LinnesLab-Passives:R0603
- removed R12, R15: 100k, LinnesLab-Passives:R0603
- removed SD2: (no value), LinnesLab-Connectors:MICROSD
- removed U5: PCF8523, LinnesLab-Clocks:SO8
- removed XTAL3: 32.7680kHz, LinnesLab-Clocks:2-SMD.NOLEAD.2.0MMTO1.2MM
- moved C24 56.1 mm to (13.8, 2.99)
- moved C25 56.1 mm to (13.8, 6.72)
- moved JP2 56.1 mm to (3.15, 3.62)
- moved LED5 56.1 mm to (14.6, 9.26)
- moved LED6 56.1 mm to (15.0, 11.5)
- moved R1 56.1 mm to (9.65, 13.8)
- moved R18 56.1 mm to (11.2, 5.96)
- moved R19 56.1 mm to (11.2, 3.65)
- moved R20 56.1 mm to (11.2, 9.24)
- moved R21 56.1 mm to (11.6, 11.6)
- moved U4 56.1 mm to (6.10, 8.32)
- moved R2 55.8 mm to (5.45, 13.7)
- moved C9 43.9 mm to (18.4, 21.8), turned to 90 degrees
- moved C8 41.6 mm to (16.9, 21.7), turned to 270 degrees
- moved XTAL2 41.2 mm to (20.0, 21.4), turned to 90 degrees
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Connections:
- removed net CD2: SD2.CD2
- removed net N$17: CHRG.5, R11.2
- removed net N$19: U5.2, XTAL3.P$1
- removed net N$20: U5.1, XTAL3.P$2
- removed net VBAT: U5.3
- net 3.3V: no longer C2.1, C6.1, LDO2.5, R15.2, SD2.4, U5.8
- net D27/CHRGSTATUS: no longer CHRG.1, R12.1
- net D5/CD1: no longer SD2.CD1
- net D7/SD.CS: no longer SD2.2
- net GND: no longer C2.2, C20.2, C21.1, C5.1, C6.2, CHRG.2, LDO2.2, R11.1, R15.1, SD2.6, SD2.MT1, SD2.MT2, U5.4
- net MISO: no longer SD2.7
- net MOSI: no longer SD2.3
- net SCK: no longer SD2.5
- net SCL: no longer U5.6
- net SDA: no longer U5.5
- net VIN: no longer C21.2, C5.2, CHRG.4, LDO2.1, LDO2.3, R12.2
- net VLIPO: no longer C20.1, CHRG.3
Routing:
- net SWO: track 0.00 -> 11.9 mm, vias 0 -> 1
- net N$4: track 0.00 -> 8.39 mm
- net SWCLK: track 0.00 -> 7.95 mm
- net LED2: track 0.00 -> 7.86 mm
- net N$6: track 0.00 -> 7.01 mm
- net GND: track 28.9 -> 35.0 mm, vias 16 -> 18
- net VLIPO: track 13.3 -> 19.1 mm
- net RESET: track 0.00 -> 5.10 mm
- net SWDIO: track 0.00 -> 5.07 mm, vias 0 -> 1
- net LED1: track 0.00 -> 5.05 mm
- net 3.3V: track 5.92 -> 1.96 mm, vias 1 -> 0
- net N$15: track 3.10 -> 1.00 mm
- net TXLED: track 12.5 -> 14.6 mm
- net A4/BATT: track 0.00 -> 1.94 mm
- net VIN: track 8.36 -> 6.47 mm
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