File: Hardware/Top/D2D-TOP.brd (EAGLE design)
At the start: 38 x 38 mm, 55 parts, among them SW1 SWITCH.MOM, SW2 SWITCH.MOM, U2 NRF52832_MODULE_MDBT42, U4 FT231XS, U6 PHOTOTRANSISTOR

Commit message: finished 006
Parts:
- moved R5 1.76 mm to (33.7, 12.9)
- moved D1 1.62 mm to (33.8, 11.3)
- moved C14 1.59 mm to (33.7, 9.85)
- moved C18 1.56 mm to (24.9, 16.2)
- moved R4 0.90 mm to (34.5, 23.4)
- moved R3 0.89 mm to (32.4, 23.4)
- moved L2 0.85 mm to (18.8, 25.9)
- moved SW4 0.84 mm to (33.7, 15.9), turned to 90 degrees
- moved C7 0.82 mm to (18.8, 29.4)
- moved LED4 0.71 mm to (34.5, 20.4)
- moved LED3 0.68 mm to (32.6, 20.4)
- moved U2 0.67 mm to (25.6, 29.7)
- moved XTAL2 0.48 mm to (19.6, 21.4)
- moved C9 0.34 mm to (18.1, 21.8)
- moved R7 0.31 mm to (31.2, 18.6)
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Routing:
- net RESET: track 5.10 -> 29.2 mm
- net SWCLK: track 7.95 -> 9.58 mm, vias 0 -> 1
- net SWO: track 11.9 -> 12.8 mm
- net SWDIO: track 5.07 -> 5.73 mm
- net N$10: track 1.76 -> 1.25 mm

Commit message: Finish Top
Parts:
- removed C4: 2.2u, LinnesLab-Passives:C0603
- removed R16: 10k, LinnesLab-Passives:R0603
- removed U6: PHOTOTRANSISTOR, LinnesLab-Sensors:R0603
- moved C11 48.2 mm to (22.9, 13.8)
- moved C23 45.9 mm to (1.64, 9.94), turned to 270 degrees
- moved C10 44.4 mm to (26.8, 13.0)
- moved SW3 14.7 mm to (34.4, 34.9), turned to 180 degrees
- moved R9 9.86 mm to (5.67, 29.8), turned to 270 degrees
- moved C12 7.95 mm to (16.6, 31.1)
- moved R8 6.94 mm to (3.62, 29.9), turned to 270 degrees
- moved C18 2.34 mm to (27.1, 15.3)
- moved L2 2.06 mm to (17.0, 26.8), turned to 0 degrees
- moved C7 2.00 mm to (16.8, 29.3), turned to 180 degrees
- moved C25 1.86 mm to (15.6, 6.79)
- moved C24 1.50 mm to (14.0, 4.49), turned to 90 degrees
- moved J2 1.11 mm to (2.53, 17.1)
- moved R7 1.04 mm to (31.0, 17.5)
- moved C16 0.94 mm to (29.6, 17.5)
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Connections:
- removed net A4/BATT: R13.1, R14.2, U2.5
- removed net A6/TIA: J1.6, U2.7
- removed net A7/PPG: J1.7, U2.8
- removed net D29/LED.CTRL: J1.5, U2.6
- removed net OUTPUT: C4.1, R16.2, U6.2
- new net A4/PPG: J1.7, U2.5
- new net A5/TIA: J1.6, U2.6
- new net A7/BATT: R13.1, R14.2, U2.8
- new net D30/LED.CTRL: J1.5, U2.7
- net 3.3V: no longer U6.1
- net GND: no longer C4.2, R16.1
Routing:
- net DTR: track 0.00 -> 41.3 mm, vias 0 -> 4
- net SCL: track 0.00 -> 25.5 mm, vias 0 -> 1
- net TXD.NRF: track 0.00 -> 25.2 mm, vias 0 -> 2
- net D15/SW2: track 0.00 -> 24.5 mm
- net GND: track 34.8 -> 57.7 mm, vias 18 -> 30
- net A7/BATT: track 0.00 -> 22.7 mm, vias 0 -> 2
- net SDA: track 0.00 -> 22.2 mm, vias 0 -> 1
- net RXD.NRF: track 0.00 -> 21.8 mm, vias 0 -> 2
- net MOSI: track 0.00 -> 20.9 mm, vias 0 -> 2
- net USB-: track 1.80 -> 22.6 mm, vias 0 -> 1
- net D11/SW1: track 0.00 -> 20.4 mm
- net D16/CS.OLED: track 0.00 -> 18.6 mm, vias 0 -> 2
- net D30/LED.CTRL: track 0.00 -> 16.6 mm, vias 0 -> 1
- net SCK: track 0.00 -> 15.8 mm, vias 0 -> 2
- net A5/TIA: track 0.00 -> 15.7 mm, vias 0 -> 1
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
Commit message: Finished Top board with modifications
Parts:
- added C3, C4: 4.7u, LinnesLab-Passives:C0603
- added C5, C6: 1u, LinnesLab-Passives:C0603
- added CHRG: MCP73831, LinnesLab-Power:SOT23-5
- added LDO2: MIC5504, LinnesLab-Power:SOT23-5
- added R10, R12: 100k, LinnesLab-Passives:R0603
- added R11: (no value), LinnesLab-Passives:R0603
- moved R9 4.35 mm to (3.37, 33.5), turned to 90 degrees
- moved R8 4.09 mm to (1.86, 33.6), turned to 90 degrees
Connections:
- new net N$16: CHRG.5, R11.2
- net 3.3V: now also C6.1, LDO2.5, R10.2
- net D27/CHRGSTATUS: now also CHRG.1, R12.1
- net GND: now also C3.2, C4.1, C5.1, C6.2, CHRG.2, LDO2.2, R10.1, R11.1
- net VIN: now also C4.2, C5.2, CHRG.4, LDO2.1, LDO2.3, R12.2
- net VLIPO: now also C3.1, CHRG.3
Routing:
- net VIN: track 1.73 -> 44.7 mm, vias 0 -> 2
- net D27/CHRGSTATUS: track 0.00 -> 29.4 mm, vias 0 -> 2
- net GND: track 57.7 -> 75.8 mm, vias 30 -> 33
- net VLIPO: track 19.9 -> 30.0 mm, vias 0 -> 1
- net 3.3V: track 2.01 -> 9.54 mm
- net N$16: track 0.00 -> 1.71 mm
- net SDA: track 22.2 -> 23.2 mm
- net SCL: track 25.5 -> 26.3 mm

Commit message: fixed up top schematic
Parts:
- removed C23: 100n, LinnesLab-Passives:C0603
- removed C24, C25: 47p, LinnesLab-Passives:C0603
- removed D4: (no value), LinnesLab-DiscreteSemi:USC
- removed LED5: RED, LinnesLab-LED:LED-0603
- removed LED6: YELLOW, LinnesLab-LED:LED-0603
- removed R19: 27, LinnesLab-Passives:R0603
- removed U4: FT231XS, LinnesLab-DigitalIC:SSOP20_L
- added C1: 1u, LinnesLab-Passives:C0603
- added C2: 10u, LinnesLab-Passives:C0805
- added C20: 100n, LinnesLab-Passives:C0603
- added D3: (no value), LinnesLab-DiscreteSemi:USC
- added LED1: RED, LinnesLab-LED:LED-0603
- added LED2: BLUE, LinnesLab-LED:LED-0603
- added R17: 0, LinnesLab-Passives:R0603
- added U1: NRF52832_MODULE_MDBT42, LinnesLab-Microcontrollers:BLE_MODULE_RAYTAC_MDBT42
- C10: value 300p -> 4.7u
- C11: value 300p -> 47p
- C12: value 10u -> 47p; device LinnesLab-Passives:C0805 -> LinnesLab-Passives:C0603
- C13: value 2.2uF -> 10uF; device LinnesLab-Passives:C0402 -> LinnesLab-Passives:C0603
- C16: value 10uF -> 2.2uF; device LinnesLab-Passives:C0603 -> LinnesLab-Passives:C0402
- C3, C4: value 4.7u -> (none)
- C5: value 1u -> 4.7u
- C6: value 1u -> 300p
- C8: value (none) -> 300p
- C9: value (none) -> 1u
- J1: device LinnesLab-Connectors:1X07_1.27MM -> LinnesLab-Connectors:1X02
- J2: device LinnesLab-Connectors:1X02 -> LinnesLab-Connectors:1X07_1.27MM
- LED4: value BLUE -> YELLOW
- R1: value 0 -> 10k
- R10, R14: value 100k -> 10k
- R11: value (none) -> 27
- R12: value 100k -> 27
- R13: value 100k -> 390k
- R18: value 27 -> 0
- R2: value 0 -> (none)
- R3: value 1k -> 100k
- R5: value 10k -> (none)
- R6, R8: value 10k -> 100k
- R7: value 390k -> 1k
- R9: value (none) -> 100k
- SW1, SW2: value SWITCH.MOM -> (none); device LinnesLab-Switches:TACTILE_SWITCH_SMD_6.2MM_TALL -> LinnesLab-Switches:BUTTON-GULLWING
- SW3, SW4: value (none) -> SWITCH.MOM; device LinnesLab-Switches:BUTTON-GULLWING -> LinnesLab-Switches:TACTILE_SWITCH_SMD_6.2MM_TALL
- U2: value NRF52832_MODULE_MDBT42 -> FT231XS; device LinnesLab-Microcontrollers:BLE_MODULE_RAYTAC_MDBT42 -> LinnesLab-DigitalIC:SSOP20_L
- moved R5 35.8 mm to (2.75, 29.8)
- moved R14 33.3 mm to (34.3, 12.8), turned to 180 degrees
- moved SW3 33.3 mm to (21.3, 4.38)
- moved C14 32.7 mm to (1.64, 9.94), turned to 270 degrees
- moved SW2 30.7 mm to (34.4, 34.9)
- moved U2 29.4 mm to (6.12, 7.69), turned to 270 degrees
- moved R3 27.8 mm to (5.94, 29.8), turned to 0 degrees
- moved R13 27.6 mm to (31.0, 17.5)
- moved C12 26.8 mm to (14.0, 4.49), turned to 90 degrees
- moved R12 26.7 mm to (11.2, 3.65), turned to 180 degrees
- moved C10 26.4 mm to (2.75, 24.0), turned to 180 degrees
- moved D1 26.3 mm to (9.07, 4.15), flipped to the bottom, turned to 270 degrees
- moved R11 25.3 mm to (11.2, 5.96)
- moved LED4 22.1 mm to (15.0, 11.5), turned to 180 degrees
- moved LED3 21.8 mm to (14.6, 9.26), turned to 180 degrees
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- renumbered CHRG to CHRG1, CORTEX1 to DEBUG1, D5 to D2, JP2 to JP1, L2 to L1, LDO2 to LDO1, R20 to R15, R21 to R16, USB2 to USB1, XTAL2 to XTAL1
Connections:
- net 3.3V: now also C14.2, C18.2, C2.2, C9.1, D3.-, J2.4, LED3.A, LED4.A, R1.2, R14.2, R2.2, R6.2, U1.11, U2.14, U2.3; no longer C12.2, C17.2, C23.2, C6.1, D1.-, J1.4, LED5.A, LED6.A, R10.2, R5.2, R8.2, R9.2, U2.11, U4.14, U4.3
- net A4/PPG: now also J2.7, U1.5; no longer J1.7, U2.5
- net A5/TIA: now also J2.6, U1.6; no longer J1.6, U2.6
- net A7/BATT: now also R8.1, R9.2, U1.8; no longer R13.1, R14.2, U2.8
- net CTS: now also U2.9; no longer U4.9
- net D11/SW1: now also SW3.A1, U1.25; no longer SW1.A1, U2.25
- net D15/SW2: now also SW4.A1, U1.29; no longer SW2.A1, U2.29
- net D16/CS.OLED: now also U1.30; no longer U2.30
- net D27/CHRGSTATUS: now also R3.1, U1.4; no longer R12.1, U2.4
- net D3/RESET.OLED: now also U1.16; no longer U2.16
- net D30/LED.CTRL: now also J2.5, U1.7; no longer J1.5, U2.7
- net D4/DC.OLED: now also U1.17; no longer U2.17
- net D5/CD1: now also U1.18; no longer U2.18
- net D7/SD.CS: now also U1.20; no longer U2.20
- net DFU: now also SW2.3, U1.34; no longer SW3.3, U2.34
- net DTR: now also C20.1, U2.1; no longer C14.1, U4.1
- net FRST: now also U1.38; no longer U2.38
- net FT3V3: now also U2.13; no longer U4.13
- net GND: now also C1.2, C11.1, C12.2, C13.1, C14.1, C2.1, C3.1, C4.2, C7.1, C8.2, J1.1, J2.3, LED1.C, LED2.C, R13.2, R5.1, R9.1, SW1.3, SW2.1, SW3.B1, SW3.B2, SW4.B1, SW4.B2, U1.1, U1.12, U1.24, U1.39, U2.16, U2.6; no longer C11.2, C12.1, C17.1, C23.1, C24.2, C25.1, C3.2, C4.1, C7.2, C8.1, J1.3, J2.1, LED3.C, LED4.C, R11.1, R14.1, R7.2, SW1.B1, SW1.B2, SW2.B1, SW2.B2, SW3.1, SW4.3, U2.1, U2.12, U2.24, U2.39, U4.16, U4.6
- net LED1: now also R4.2, U1.31; no longer R3.2, U2.31
- net LED2: now also R7.2, U1.33; no longer R4.2, U2.33
- net MISO: now also U1.28; no longer U2.28
- net MOSI: now also U1.27; no longer U2.27
- net N$1: now also R10.2; no longer R6.2
- net N$10: now also LED2.A, R7.1; no longer LED4.A, R4.1
- net N$11: now also U1.10; no longer U2.10
- net N$12: now also C1.1, U1.9; no longer C7.1, U2.9
- net N$13: now also C13.2; no longer C16.2
- net N$15: now also C16.2; no longer C18.2
- net N$16: now also R5.2; no longer R11.2
- net N$2: now also R13.1; no longer R7.1
- net N$23: now also R11.2, U2.12; no longer R18.2, U4.12
- net N$24: now also R12.2, U2.11; no longer R19.2, U4.11
- net N$25: now also LED3.C; no longer LED5.C
- net N$26: now also LED4.C; no longer LED6.C
- net N$3: now also C17.2; no longer C13.2
- net N$4: now also C3.2, U1.13; no longer C8.2, U2.13
- net N$5: now also C17.1; no longer C13.1
- net N$6: now also C4.1, U1.14; no longer C9.1, U2.14
- net N$9: now also LED1.A, R4.1; no longer LED3.A, R3.1
- net P0.09/NFC1: now also C6.1, U1.22; no longer C11.1, U2.22
- net P0.10/NFC2: now also C8.1, U1.23; no longer C10.1, U2.23
- net RESET: now also C20.2, D3.+, R14.1, SW1.1, U1.35; no longer C14.2, D1.+, R5.1, SW4.1, U2.35
- net RXD.FT: now also R18.1, U2.4; no longer R2.1, U4.4
- net RXD.NRF: now also R17.2, U1.21; no longer R1.2, U2.21
- net RXLED: now also U2.17; no longer U4.17
- net SCK: now also U1.26; no longer U2.26
- net SCL: now also J2.2, R2.1, U1.3; no longer J1.2, R9.1, U2.3
- net SDA: now also J2.1, R1.1, U1.2; no longer J1.1, R8.1, U2.2
- net SWCLK: now also U1.36; no longer U2.36
- net SWDIO: now also U1.37; no longer U2.37
- net SWO: now also U1.32; no longer U2.32
- net TXD.FT: now also R17.1, U2.20; no longer R1.1, U4.20
- net TXD.NRF: now also R18.2, U1.19; no longer R2.2, U2.19
- net TXLED: now also U2.10; no longer U4.10
- net USB+: now also C12.1, R12.1; no longer C24.1, R19.1
- net USB-: now also C11.2, R11.1; no longer C25.2, R18.1
- net VIN: now also C7.2, D1.-, R3.2; no longer C4.2, D4.-, R12.2
- net VLIPO: now also C10.1, D1.+, J1.2, R8.2; no longer C3.1, D4.+, J2.2, R13.2
- net V_USB: now also U2.15; no longer U4.15
Other:
- board text added: "+"
