File: Hardware/Top/D2D-TOP.sch (EAGLE design)
At the start: 69 parts, among them SW1 SWITCH.MOM, SW2 SWITCH.MOM, U2 NRF52832_MODULE_MDBT42, U4 PCF8523, U5 FT231XS, U6 PHOTOTRANSISTOR

Commit message: updated top board
Parts:
- U4: value PCF8523 -> FT231XS; device LinnesLab-Clocks:PCF8523 -> LinnesLab-DigitalIC:FT231XS; DIGIKEY 568-5306-1-ND -> (none); I2C_ADDRESS 0x68h -> (none); MFN PCF8523T/1,118 -> (none); MFN_MANUFACTURER NXP USA Inc. -> (none)
- U5: value FT231XS -> PCF8523; device LinnesLab-DigitalIC:FT231XS -> LinnesLab-Clocks:PCF8523; DIGIKEY (none) -> 568-5306-1-ND; I2C_ADDRESS (none) -> 0x68h; MFN (none) -> PCF8523T/1,118; MFN_MANUFACTURER (none) -> NXP USA Inc.
Connections:
- net 3.3V: now also U4.!RESET, U4.VCCIO, U5.VDD; no longer U4.VDD, U5.!RESET, U5.VCCIO
- net CTS: now also U4.!CTS; no longer U5.!CTS
- net DTR: now also U4.!DTR; no longer U5.!DTR
- net FT3V3: now also U4.3V3OUT; no longer U5.3V3OUT
- net GND: now also U4.GND@16, U4.GND@6, U5.VSS; no longer U4.VSS, U5.GND@16, U5.GND@6
- net N$19: now also U5.OSCO; no longer U4.OSCO
- net N$20: now also U5.OSCI; no longer U4.OSCI
- net N$23: now also U4.USBDM; no longer U5.USBDM
- net N$24: now also U4.USBDP; no longer U5.USBDP
- net RXD.FT: now also U4.RXD; no longer U5.RXD
- net RXLED: now also U4.CBUS1; no longer U5.CBUS1
- net SCL: now also U5.SCL; no longer U4.SCL
- net SDA: now also U5.SDA; no longer U4.SDA
- net TXD.FT: now also U4.TXD; no longer U5.TXD
- net TXLED: now also U4.CBUS2; no longer U5.CBUS2
- net V_USB: now also U4.VCC; no longer U5.VCC
Other:
- moved on the sheet: R1, R2
Changed lines of the file:
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@@
 <attribute name="FREQ" value="32.7680KHZ"/>
 </part>
-<part name="U4" library="LinnesLab-Clocks" deviceset="PCF8523" device="" package3d_urn="urn:adsk.eagle:package:18599600/2">
+<part name="U5" library="LinnesLab-Clocks" deviceset="PCF8523" device="" package3d_urn="urn:adsk.eagle:package:18599600/2">
 <attribute name="DIGIKEY" value="568-5306-1-ND"/>
 <attribute name="I2C_ADDRESS" value="0x68h"/>
@@
 <part name="GND49" library="LinnesLab-Symbols" deviceset="GND" device=""/>
 <part name="GND50" library="LinnesLab-Symbols" deviceset="GND" device=""/>
-<part name="U5" library="LinnesLab-DigitalIC" deviceset="FT231X" device="S"/>
+<part name="U4" library="LinnesLab-DigitalIC" deviceset="FT231X" device="S"/>
 <part name="R1" library="LinnesLab-Passives" deviceset="RESISTOR" device="0603" package3d_urn="urn:adsk.eagle:package:15661944/2" value="0"/>
 <part name="R2" library="LinnesLab-Passives" deviceset="RESISTOR" device="0603" package3d_urn="urn:adsk.eagle:package:15661944/2" value="0"/>
@@
 <attribute name="FREQ" x="279.4" y="-12.7" size="1.27" layer="96" display="off"/>
 </instance>
-<instance part="U4" gate="G$1" x="299.72" y="-15.24" smashed="yes">
+<instance part="U5" gate="G$1" x="299.72" y="-15.24" smashed="yes">
 <attribute name="NAME" x="287.02" y="-8.89" size="1.778" layer="95"/>
 <attribute name="VALUE" x="287.02" y="-25.4" size="1.778" layer="96"/>
@@
 <attribute name="VALUE" x="243.84" y="223.266" size="1.778" layer="96" align="top-center"/>
 </instance>
-<instance part="U5" gate="U$1" x="292.1" y="238.76" smashed="yes">
+<instance part="U4" gate="U$1" x="292.1" y="238.76" smashed="yes">
 <attribute name="NAME" x="281.94" y="256.794" size="1.778" layer="95"/>
 <attribute name="VALUE" x="281.94" y="220.472" size="1.778" layer="96" align="top-left"/>
 </instance>
-<instance part="R1" gate="G$1" x="353.06" y="254" smashed="yes">
-<attribute name="NAME" x="349.25" y="258.0386" size="1.778" layer="95"/>
-<attribute name="VALUE" x="349.25" y="250.698" size="1.778" layer="96"/>
-</instance>
-<instance part="R2" gate="G$1" x="355.6" y="243.84" smashed="yes">
-<attribute name="NAME" x="354.33" y="245.3386" size="1.778" layer="95"/>
-<attribute name="VALUE" x="351.79" y="240.538" size="1.778" layer="96"/>
+<instance part="R1" gate="G$1" x="360.68" y="254" smashed="yes">
+<attribute name="NAME" x="356.87" y="258.0386" size="1.778" layer="95"/>
+<attribute name="VALUE" x="356.87" y="250.698" size="1.778" layer="96"/>
+</instance>
+<instance part="R2" gate="G$1" x="363.22" y="243.84" smashed="yes">
+<attribute name="NAME" x="361.95" y="245.3386" size="1.778" layer="95"/>
+<attribute name="VALUE" x="359.41" y="240.538" size="1.778" layer="96"/>
 </instance>
 <instance part="R8" gate="G$1" x="-25.4" y="162.56" smashed="yes" rot="R90">
@@
 <wire x1="281.94" y1="-22.86" x2="281.94" y2="-20.32" width="0.1524" layer="91"/>
 <pinref part="GND3" gate="G$1" pin="GND"/>
-<pinref part="U4" gate="G$1" pin="VSS"/>
+<pinref part="U5" gate="G$1" pin="VSS"/>
 </segment>
 <segment>
@@
 <junction x="276.86" y="223.52"/>
 <pinref part="GND46" gate="G$1" pin="GND"/>
-<pinref part="U5" gate="U$1" pin="GND@6"/>
-<pinref part="U5" gate="U$1" pin="GND@16"/>
+<pinref part="U4" gate="U$1" pin="GND@6"/>
+<pinref part="U4" gate="U$1" pin="GND@16"/>
 </segment>
 <segment>
@@
 <wire x1="317.5" y1="-10.16" x2="317.5" y2="-12.7" width="0.1524" layer="91"/>
 <pinref part="SUPPLY10" gate="G$1" pin="3.3V"/>
-<pinref part="U4" gate="G$1" pin="VDD"/>
+<pinref part="U5" gate="G$1" pin="VDD"/>
 </segment>
 <segment>
@@
 <wire x1="279.4" y1="236.22" x2="269.24" y2="236.22" width="0.1524" layer="91"/>
 <junction x="269.24" y="236.22"/>
-<pinref part="U5" gate="U$1" pin="VCCIO"/>
-<pinref part="U5" gate="U$1" pin="!RESET"/>
+<pinref part="U4" gate="U$1" pin="VCCIO"/>
+<pinref part="U4" gate="U$1" pin="!RESET"/>
 </segment>
 <segment>
@@
 <wire x1="314.96" y1="-20.32" x2="335.28" y2="-20.32" width="0.1524" layer="91"/>
 <label x="335.28" y="-20.32" size="1.27" layer="95" xref="yes"/>
-<pinref part="U4" gate="G$1" pin="SDA"/>
+<pinref part="U5" gate="G$1" pin="SDA"/>
 </segment>
 <segment>
@@
 <label x="335.28" y="-17.78" size="1.27" layer="95" xref="yes"/>
 <wire x1="314.96" y1="-17.78" x2="335.28" y2="-17.78" width="0.1524" layer="91"/>
-<pinref part="U4" gate="G$1" pin="SCL"/>
+<pinref part="U5" gate="G$1" pin="SCL"/>
 </segment>
 <segment>
@@
 <wire x1="304.8" y1="241.3" x2="309.88" y2="241.3" width="0.1524" layer="91"/>
 <label x="309.88" y="241.3" size="1.27" layer="95" xref="yes"/>
-<pinref part="U5" gate="U$1" pin="!DTR"/>
+<pinref part="U4" gate="U$1" pin="!DTR"/>
 </segment>
 </net>
@@
 <wire x1="276.86" y1="254" x2="276.86" y2="259.08" width="0.1524" layer="91"/>
 <pinref part="SUPPLY22" gate="G$1" pin="V_USB"/>
-<pinref part="U5" gate="U$1" pin="VCC"/>
+<pinref part="U4" gate="U$1" pin="VCC"/>
 </segment>
 </net>
@@
 <wire x1="274.32" y1="-12.7" x2="276.86" y2="-12.7" width="0.1524" layer="91"/>
 <pinref part="XTAL3" gate="G$1" pin="1"/>
-<pinref part="U4" gate="G$1" pin="OSCO"/>
+<pinref part="U5" gate="G$1" pin="OSCO"/>
 </segment>
 </net>
@@
 <wire x1="281.94" y1="-12.7" x2="284.48" y2="-12.7" width="0.1524" layer="91"/>
 <pinref part="XTAL3" gate="G$1" pin="2"/>
-<pinref part="U4" gate="G$1" pin="OSCI"/>
+<pinref part="U5" gate="G$1" pin="OSCI"/>
 </segment>
 </net>
@@
 <wire x1="279.4" y1="243.84" x2="266.7" y2="243.84" width="0.1524" layer="91"/>
 <pinref part="R18" gate="G$1" pin="2"/>
-<pinref part="U5" gate="U$1" pin="USBDM"/>
+<pinref part="U4" gate="U$1" pin="USBDM"/>
 </segment>
 </net>
@@
 <wire x1="279.4" y1="241.3" x2="266.7" y2="241.3" width="0.1524" layer="91"/>
 <pinref part="R19" gate="G$1" pin="2"/>
-<pinref part="U5" gate="U$1" pin="USBDP"/>
+<pinref part="U4" gate="U$1" pin="USBDP"/>
 </segment>
 </net>
@@
 <pinref part="JP2" gate="G$1" pin="2"/>
 <label x="307.34" y="243.84" size="1.27" layer="95" xref="yes"/>
-<pinref part="U5" gate="U$1" pin="!CTS"/>
+<pinref part="U4" gate="U$1" pin="!CTS"/>
 </segment>
 </net>
@@
 <wire x1="322.58" y1="228.6" x2="322.58" y2="236.22" width="0.1524" layer="91"/>
 <label x="312.42" y="228.6" size="1.27" layer="95"/>
-<pinref part="U5" gate="U$1" pin="CBUS1"/>
+<pinref part="U4" gate="U$1" pin="CBUS1"/>
 </segment>
 </net>
@@
 <wire x1="332.74" y1="226.06" x2="332.74" y2="236.22" width="0.1524" layer="91"/>
 <label x="312.42" y="226.06" size="1.27" layer="95"/>
-<pinref part="U5" gate="U$1" pin="CBUS2"/>
+<pinref part="U4" gate="U$1" pin="CBUS2"/>
 </segment>
 </net>
 <net name="FT3V3" class="0">
 <segment>
-<pinref part="U5" gate="U$1" pin="3V3OUT"/>
+<pinref part="U4" gate="U$1" pin="3V3OUT"/>
 <wire x1="279.4" y1="248.92" x2="276.86" y2="248.92" width="0.1524" layer="91"/>
 <label x="276.86" y="248.92" size="1.27" layer="95" rot="R180" xref="yes"/>
@@
 <wire x1="307.34" y1="254" x2="304.8" y2="254" width="0.1524" layer="91"/>
 <label x="307.34" y="254" size="1.27" layer="95" xref="yes"/>
-<pinref part="U5" gate="U$1" pin="TXD"/>
+<pinref part="U4" gate="U$1" pin="TXD"/>
 </segment>
 <segment>
 <pinref part="R1" gate="G$1" pin="1"/>
-<wire x1="347.98" y1="254" x2="345.44" y2="254" width="0.1524" layer="91"/>
-<label x="345.44" y="254" size="1.27" layer="95" rot="R180" xref="yes"/>
+<wire x1="355.6" y1="254" x2="353.06" y2="254" width="0.1524" layer="91"/>
+<label x="353.06" y="254" size="1.27" layer="95" rot="R180" xref="yes"/>
 </segment>
 </net>
@@
 <segment>
 <pinref part="R1" gate="G$1" pin="2"/>
-<wire x1="358.14" y1="254" x2="363.22" y2="254" width="0.1524" layer="91"/>
-<label x="363.22" y="254" size="1.27" layer="95" xref="yes"/>
+<wire x1="365.76" y1="254" x2="370.84" y2="254" width="0.1524" layer="91"/>
+<label x="370.84" y="254" size="1.27" layer="95" xref="yes"/>
 </segment>
 <segment>
@@
 <segment>
 <pinref part="R2" gate="G$1" pin="2"/>
-<wire x1="360.68" y1="243.84" x2="363.22" y2="243.84" width="0.1524" layer="91"/>
-<label x="363.22" y="243.84" size="1.27" layer="95" xref="yes"/>
+<wire x1="368.3" y1="243.84" x2="370.84" y2="243.84" width="0.1524" layer="91"/>
+<label x="370.84" y="243.84" size="1.27" layer="95" xref="yes"/>
 </segment>
 <segment>
@@
 <segment>
 <pinref part="R2" gate="G$1" pin="1"/>
-<wire x1="350.52" y1="243.84" x2="347.98" y2="243.84" width="0.1524" layer="91"/>
-<label x="347.98" y="243.84" size="1.27" layer="95" rot="R180" xref="yes"/>
+<wire x1="358.14" y1="243.84" x2="355.6" y2="243.84" width="0.1524" layer="91"/>
+<label x="355.6" y="243.84" size="1.27" layer="95" rot="R180" xref="yes"/>
 </segment>
 <segment>
 <wire x1="307.34" y1="251.46" x2="304.8" y2="251.46" width="0.1524" layer="91"/>
 <label x="307.34" y="251.46" size="1.27" layer="95" xref="yes"/>
-<pinref part="U5" gate="U$1" pin="RXD"/>
-</segment>
-</net>
+<pinref part="U4" gate="U$1" pin="RXD"/>
+</segment>
+</net>

Commit message: completed 004
Parts:
- removed GPS.PWR: MIC5504, LinnesLab-Power:MIC5504
Connections:
- removed net D2/GPS.PWR: GPS.PWR.EN, U2.P0.02/AIN0
Changed lines of the file:
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@@
 <part name="SUPPLY8" library="LinnesLab-Symbols" deviceset="3.3V" device=""/>
 <part name="GND5" library="LinnesLab-Symbols" deviceset="GND" device=""/>
-<part name="GPS.PWR" library="LinnesLab-Power" deviceset="MIC5504" device=""/>
 </parts>
 <sheets>
@@
 <attribute name="VALUE" x="20.32" y="230.886" size="1.778" layer="96" align="top-center"/>
 </instance>
-<instance part="GPS.PWR" gate="G$1" x="137.16" y="-5.08" smashed="yes">
-<attribute name="NAME" x="129.54" y="3.81" size="1.778" layer="95"/>
-<attribute name="VALUE" x="129.54" y="-15.24" size="1.778" layer="96"/>
-</instance>
 </instances>
 <busses>
@@
 </segment>
 </net>
-<net name="D2/GPS.PWR" class="0">
-<segment>
-<pinref part="U2" gate="G$1" pin="P0.02/AIN0"/>
-<wire x1="53.34" y1="88.9" x2="53.34" y2="86.36" width="0.1524" layer="91"/>
-<label x="53.34" y="86.36" size="1.27" layer="95" rot="R270" xref="yes"/>
-</segment>
-<segment>
-<pinref part="GPS.PWR" gate="G$1" pin="EN"/>
-<wire x1="127" y1="-10.16" x2="124.46" y2="-10.16" width="0.1524" layer="91"/>
-<label x="124.46" y="-10.16" size="1.27" layer="95" rot="R180" xref="yes"/>
-</segment>
-</net>

Commit message: push onto repo
Parts:
- removed C2, C5, C6: 1u, LinnesLab-Passives:CAPACITOR0603
- removed C20, C21: 4.7u, LinnesLab-Passives:CAPACITOR0603
- removed CHRG: MCP73831, LinnesLab-Power:MCP73831
- removed LDO2: MIC5504, LinnesLab-Power:MIC5504
- removed R11: (no value), LinnesLab-Passives:RESISTOR0603
- removed R12, R15: 100k, LinnesLab-Passives:RESISTOR0603
- removed SD2: (no value), LinnesLab-Connectors:MICROSD
- removed U5: PCF8523, LinnesLab-Clocks:PCF8523
- removed XTAL3: 32.7680kHz, LinnesLab-Clocks:CRYSTALECS-.327-12.5-12-C-TR
Connections:
- removed net CD2: SD2.CARD_DETECT1
- removed net N$17: CHRG.PROG, R11.2
- removed net N$19: U5.OSCO, XTAL3.1
- removed net N$20: U5.OSCI, XTAL3.2
- net 3.3V: no longer C2.1, C6.1, LDO2.OUT, R15.2, SD2.VDD, U5.VDD
- net D27/CHRGSTATUS: no longer CHRG.STAT, R12.1
- net D5/CD1: no longer SD2.CARD_DETECT
- net D7/SD.CS: no longer SD2.CS
- net GND: no longer C2.2, C20.2, C21.1, C5.1, C6.2, CHRG.VSS, LDO2.GND, R11.1, R15.1, SD2.GND, SD2.GND1, SD2.VSS, U5.VSS
- net MISO: no longer SD2.DATA_OUT
- net MOSI: no longer SD2.DATA_IN
- net SCK: no longer SD2.SCLK
- net SCL: no longer U5.SCL
- net SDA: no longer U5.SDA
- net VIN: no longer C21.2, C5.2, CHRG.VIN, LDO2.EN, LDO2.IN, R12.2
- net VLIPO: no longer C20.1, CHRG.VBAT
Other:
- note removed: "Back-up battery if desired"
- note removed: "Connect MISO, MOSI, and SCK to appropriate pins on microcontroller. Those are SPI pins and are generally prespecified. You have more flexibility with the SD.CS pin."
- note removed: "I2C Address = 0x68h"
- note removed: "Real-Time Clock"
- note removed: "SD Card"
