File: Hardware/Top/D2D-TOP.sch (EAGLE design)
At the start: 55 parts, among them SW1 SWITCH.MOM, SW2 SWITCH.MOM, U2 NRF52832_MODULE_MDBT42, U4 FT231XS, U6 PHOTOTRANSISTOR

Commit message: Finish Top
Parts:
- removed C4: 2.2u, LinnesLab-Passives:CAPACITOR0603
- removed R16: 10k, LinnesLab-Passives:RESISTOR0603
- removed U6: PHOTOTRANSISTOR, LinnesLab-Sensors:PHOTOTRANSISTOR
Connections:
- removed net A4/BATT: R13.1, R14.2, U2.P0.28/AIN4
- removed net A6/TIA: J1.6, U2.P0.30/AIN6
- removed net A7/PPG: J1.7, U2.P0.31/AIN7
- removed net D29/LED.CTRL: J1.5, U2.P0.29/AIN5
- removed net OUTPUT: C4.1, R16.2, U6.E
- new net A4/PPG: J1.7, U2.P0.28/AIN4
- new net A5/TIA: J1.6, U2.P0.29/AIN5
- new net A7/BATT: R13.1, R14.2, U2.P0.31/AIN7
- new net D30/LED.CTRL: J1.5, U2.P0.30/AIN6
- net 3.3V: no longer U6.C
- net GND: no longer C4.2, R16.1
Other:
- note removed: "Ambient Light"
- note removed: "Outputs a voltage relative to incident light. Will need to calibrate RL to based on the desired dynamic range."

Commit message: Finished Top board with modifications
Parts:
- added C3, C4: 4.7u, LinnesLab-Passives:CAPACITOR0603
- added C5, C6: 1u, LinnesLab-Passives:CAPACITOR0603
- added CHRG: MCP73831, LinnesLab-Power:MCP73831
- added LDO2: MIC5504, LinnesLab-Power:MIC5504
- added R10, R12: 100k, LinnesLab-Passives:RESISTOR0603
- added R11: (no value), LinnesLab-Passives:RESISTOR0603
Connections:
- new net N$16: CHRG.PROG, R11.2
- net 3.3V: now also C6.1, LDO2.OUT, R10.2
- net D27/CHRGSTATUS: now also CHRG.STAT, R12.1
- net GND: now also C3.2, C4.1, C5.1, C6.2, CHRG.VSS, LDO2.GND, R10.1, R11.1
- net VIN: now also C4.2, C5.2, CHRG.VIN, LDO2.EN, LDO2.IN, R12.2
- net VLIPO: now also C3.1, CHRG.VBAT

Commit message: fixed up top schematic
Other:
- note added: "0 ohm Resistors in case I mixed up TX/RX like I usually do"
- note added: "D2D Basic Top Revision A Date: Saturday, 7/11/2019 Author: Alice Ding"
- note added: "Diodes switch from LiPo power to USB when USB is connected. The USB power then charges the battery"
- note added: "Headers connecting top and bottom board"
- note added: "R11 sets charge current I_charge = 1000V/R11 per MCP73831 datasheet"
- note added: "Voltage divider used to monitor battery voltage"
- note removed: "RTC"
- moved on the sheet: C10, C11, C12, C13, C14, C15, C16, C17, C18, C19, C3, C4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

Commit message: fixed up top schematic
Parts:
- removed C23: 100n, LinnesLab-Passives:CAPACITOR0603
- removed C24, C25: 47p, LinnesLab-Passives:CAPACITOR0603
- removed D4: (no value), LinnesLab-DiscreteSemi:SCHOTTKY-USC
- removed LED5: RED, LinnesLab-LED:LED0603
- removed LED6: YELLOW, LinnesLab-LED:LED0603
- removed R19: 27, LinnesLab-Passives:RESISTOR0603
- removed U4: FT231XS, LinnesLab-DigitalIC:FT231XS
- added C1: 1u, LinnesLab-Passives:CAPACITOR0603
- added C2: 10u, LinnesLab-Passives:CAPACITOR0805
- added C20: 100n, LinnesLab-Passives:CAPACITOR0603
- added D3: (no value), LinnesLab-DiscreteSemi:SCHOTTKY-USC
- added LED1: RED, LinnesLab-LED:LED0603
- added LED2: BLUE, LinnesLab-LED:LED0603
- added R17: 0, LinnesLab-Passives:RESISTOR0603
- added U1: NRF52832_MODULE_MDBT42, LinnesLab-Microcontrollers:NRF52832_MODULE_MDBT42
- C10: value 300p -> 4.7u
- C11: value 300p -> 47p
- C12: value 10u -> 47p; device LinnesLab-Passives:CAPACITOR0805 -> LinnesLab-Passives:CAPACITOR0603
- C13: value 2.2uF -> 10uF; device LinnesLab-Passives:CAPACITOR0402 -> LinnesLab-Passives:CAPACITOR0603
- C16: value 10uF -> 2.2uF; device LinnesLab-Passives:CAPACITOR0603 -> LinnesLab-Passives:CAPACITOR0402
- C3, C4: value 4.7u -> (none)
- C5: value 1u -> 4.7u
- C6: value 1u -> 300p
- C8: value (none) -> 300p
- C9: value (none) -> 1u
- J1: device LinnesLab-Connectors:CONN_07-1.27MM -> LinnesLab-Connectors:CONN_02
- J2: device LinnesLab-Connectors:CONN_02 -> LinnesLab-Connectors:CONN_07-1.27MM
- LED4: value BLUE -> YELLOW
- R1: value 0 -> 10k
- R10, R14: value 100k -> 10k
- R11: value (none) -> 27
- R12: value 100k -> 27
- R13: value 100k -> 390k
- R18: value 27 -> 0
- R2: value 0 -> (none)
- R3: value 1k -> 100k
- R5: value 10k -> (none)
- R6, R8: value 10k -> 100k
- R7: value 390k -> 1k
- R9: value (none) -> 100k
- SW1, SW2: value SWITCH.MOM -> (none); device LinnesLab-Switches:SWITCH.MOM -> LinnesLab-Switches:SPST-PTS830GG140-COPY.1-3
- SW3, SW4: value (none) -> SWITCH.MOM; device LinnesLab-Switches:SPST-PTS830GG140-COPY.1-3 -> LinnesLab-Switches:SWITCH.MOM
- U2: value NRF52832_MODULE_MDBT42 -> FT231XS; device LinnesLab-Microcontrollers:NRF52832_MODULE_MDBT42 -> LinnesLab-DigitalIC:FT231XS
- renumbered CHRG to CHRG1, CORTEX1 to DEBUG1, D5 to D2, JP2 to JP1, L2 to L1, LDO2 to LDO1, R20 to R15, R21 to R16, USB2 to USB1, XTAL2 to XTAL1
Connections:
- net 3.3V: now also C14.2, C18.2, C2.2, C9.1, D3.C, J2.4, LED3.A, LED4.A, R1.2, R14.2, R2.2, R6.2, U1.VDD, U2.!RESET, U2.VCCIO; no longer C12.2, C17.2, C23.2, C6.1, D1.C, J1.4, LED5.A, LED6.A, R10.2, R5.2, R8.2, R9.2, U2.VDD, U4.!RESET, U4.VCCIO
- net A4/PPG: now also J2.7, U1.P0.28/AIN4; no longer J1.7, U2.P0.28/AIN4
- net A5/TIA: now also J2.6, U1.P0.29/AIN5; no longer J1.6, U2.P0.29/AIN5
- net A7/BATT: now also R8.1, R9.2, U1.P0.31/AIN7; no longer R13.1, R14.2, U2.P0.31/AIN7
- net CTS: now also U2.!CTS; no longer U4.!CTS
- net D11/SW1: now also SW3.1, U1.P0.11; no longer SW1.1, U2.P0.11
- net D15/SW2: now also SW4.1, U1.P0.15; no longer SW2.1, U2.P0.15
- net D16/CS.OLED: now also U1.P0.16; no longer U2.P0.16
- net D27/CHRGSTATUS: now also R3.1, U1.P0.27; no longer R12.1, U2.P0.27
- net D3/RESET.OLED: now also U1.P0.03/AIN1; no longer U2.P0.03/AIN1
- net D30/LED.CTRL: now also J2.5, U1.P0.30/AIN6; no longer J1.5, U2.P0.30/AIN6
- net D4/DC.OLED: now also U1.P0.04/AIN2; no longer U2.P0.04/AIN2
- net D5/CD1: now also U1.P0.05/AIN3; no longer U2.P0.05/AIN3
- net D7/SD.CS: now also U1.P0.07; no longer U2.P0.07
- net DFU: now also SW2.B, U1.P0.20; no longer SW3.B, U2.P0.20
- net DTR: now also C20.1, U2.!DTR; no longer C14.1, U4.!DTR
- net FRST: now also U1.P0.22; no longer U2.P0.22
- net FT3V3: now also U2.3V3OUT; no longer U4.3V3OUT
- net GND: now also C1.2, C11.1, C12.2, C13.1, C14.1, C2.1, C3.1, C4.2, C7.1, C8.2, J1.1, J2.3, LED1.C, LED2.C, R13.2, R5.1, R9.1, SW1.B, SW2.A, SW3.3, SW3.4, SW4.3, SW4.4, U1.GND@1, U1.GND@2, U1.GND@3, U1.GND@4, U2.GND@16, U2.GND@6; no longer C11.2, C12.1, C17.1, C23.1, C24.2, C25.1, C3.2, C4.1, C7.2, C8.1, J1.3, J2.1, LED3.C, LED4.C, R11.1, R14.1, R7.2, SW1.3, SW1.4, SW2.3, SW2.4, SW3.A, SW4.B, U2.GND@1, U2.GND@2, U2.GND@3, U2.GND@4, U4.GND@16, U4.GND@6
- net LED1: now also R4.2, U1.P0.17; no longer R3.2, U2.P0.17
- net LED2: now also R7.2, U1.P0.19; no longer R4.2, U2.P0.19
- net MISO: now also U1.P0.14; no longer U2.P0.14
- net MOSI: now also U1.P0.13; no longer U2.P0.13
- net N$1: now also R10.2; no longer R6.2
- net N$10: now also LED2.A, R7.1; no longer LED4.A, R4.1
- net N$11: now also U1.DCC; no longer U2.DCC
- net N$12: now also C1.1, U1.DEC4; no longer C7.1, U2.DEC4
- net N$13: now also C13.2; no longer C16.2
- net N$15: now also C16.2; no longer C18.2
- net N$16: now also R5.2; no longer R11.2
- net N$2: now also R13.1; no longer R7.1
- net N$23: now also R11.2, U2.USBDM; no longer R18.2, U4.USBDM
- net N$24: now also R12.2, U2.USBDP; no longer R19.2, U4.USBDP
- net N$25: now also LED3.C; no longer LED5.C
- net N$26: now also LED4.C; no longer LED6.C
- net N$3: now also C17.2; no longer C13.2
- net N$4: now also C3.2, U1.P0.00/XL1; no longer C8.2, U2.P0.00/XL1
- net N$5: now also C17.1; no longer C13.1
- net N$6: now also C4.1, U1.P0.01/XL2; no longer C9.1, U2.P0.01/XL2
- net N$9: now also LED1.A, R4.1; no longer LED3.A, R3.1
- net P0.09/NFC1: now also C6.1, U1.P0.09; no longer C11.1, U2.P0.09
- net P0.10/NFC2: now also C8.1, U1.P0.10; no longer C10.1, U2.P0.10
- net RESET: now also C20.2, D3.A, R14.1, SW1.A, U1.P0.21/RESET; no longer C14.2, D1.A, R5.1, SW4.A, U2.P0.21/RESET
- net RXD.FT: now also R18.1, U2.RXD; no longer R2.1, U4.RXD
- net RXD.NRF: now also R17.2, U1.P0.08; no longer R1.2, U2.P0.08
- net RXLED: now also U2.CBUS1; no longer U4.CBUS1
- net SCK: now also U1.P0.12; no longer U2.P0.12
- net SCL: now also J2.2, R2.1, U1.P0.26; no longer J1.2, R9.1, U2.P0.26
- net SDA: now also J2.1, R1.1, U1.P0.25; no longer J1.1, R8.1, U2.P0.25
- net SWCLK: now also U1.SWDCLK; no longer U2.SWDCLK
- net SWDIO: now also U1.SWDIO; no longer U2.SWDIO
- net SWO: now also U1.P0.18/SWO; no longer U2.P0.18/SWO
- net TXD.FT: now also R17.1, U2.TXD; no longer R1.1, U4.TXD
- net TXD.NRF: now also R18.2, U1.P0.06; no longer R2.2, U2.P0.06
- net TXLED: now also U2.CBUS2; no longer U4.CBUS2
- net USB+: now also C12.1, R12.1; no longer C24.1, R19.1
- net USB-: now also C11.2, R11.1; no longer C25.2, R18.1
- net VIN: now also C7.2, D1.C, R3.2; no longer C4.2, D4.C, R12.2
- net VLIPO: now also C10.1, D1.A, J1.2, R8.2; no longer C3.1, D4.A, J2.2, R13.2
- net V_USB: now also U2.VCC; no longer U4.VCC
Other:
- moved on the sheet: C10, C11, C12, C13, C14, C16, C17, C18, C19, C3, C4, C5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
