File: Hardware/Bottom/D2D-BOTTOM.brd (EAGLE design)
At the start: 33 x 33 mm, 31 parts, among them U1 AD5242-SO16

Commit message: unfinished 002
Parts:
- added J1: (no value), LinnesLab-Connectors:1X07
- moved IMU1 17.6 mm to (9.68, 13.7)
Changed lines of the file:
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@@
 <element name="U$4" library="LinnesLab-DigitalIC" package="SOT-23-8" package3d_urn="urn:adsk.eagle:package:17879439/2" value="AD5171" x="8.5852" y="5.1054" smashed="yes">
 <attribute name="NAME" x="5.5852" y="6.8054" size="0.6604" layer="25"/>
-<attribute name="VALUE" x="5.6852" y="2.1054" size="0.6604" layer="27"/>
+<attribute name="VALUE" x="8.1998" y="35.1" size="0.6604" layer="27"/>
 </element>
 <element name="R13" library="LinnesLab-Passives" package="R0603" package3d_urn="urn:adsk.eagle:package:15661944/2" value="220k" x="10.9728" y="22.9108" smashed="yes">
@@
 <element name="C15" library="LinnesLab-Passives" package="C0603" value="2.2u" x="13.3604" y="28.4734" smashed="yes" rot="R270">
 <attribute name="NAME" x="13.9954" y="29.1084" size="0.6604" layer="25" rot="R270"/>
-<attribute name="VALUE" x="11.4554" y="29.1084" size="1.27" layer="27" rot="R270"/>
+<attribute name="VALUE" x="11.2268" y="29.591" size="1.27" layer="27" rot="R270"/>
 </element>
 <element name="C16" library="LinnesLab-Passives" package="C0603" value="2.2u" x="15.4432" y="16.4846" smashed="yes">
@@
 <attribute name="VALUE" x="36.195" y="3.175" size="1.27" layer="27"/>
 </element>
-<element name="IMU1" library="LinnesLab-Sensors" package="LSM6DS3_CAST" value="LSM6DS3_CAST" x="8.7376" y="31.3182" smashed="yes">
-<attribute name="NAME" x="6.1976" y="34.4932" size="0.6604" layer="25"/>
-<attribute name="VALUE" x="6.1976" y="26.8732" size="0.6604" layer="27"/>
+<element name="IMU1" library="LinnesLab-Sensors" package="LSM6DS3_CAST" value="LSM6DS3_CAST" x="9.6774" y="13.716" smashed="yes">
+<attribute name="NAME" x="7.1374" y="16.891" size="0.6604" layer="25"/>
+<attribute name="VALUE" x="7.1374" y="9.271" size="0.6604" layer="27"/>
 </element>
 <element name="C24" library="LinnesLab-Passives" package="C0603" value="100n" x="4.0386" y="31.0642" smashed="yes" rot="R270">
 <attribute name="NAME" x="4.6736" y="31.6992" size="0.6604" layer="25" rot="R270"/>
 <attribute name="VALUE" x="2.1336" y="31.6992" size="0.6604" layer="27" rot="R270"/>
+</element>
+<element name="J1" library="LinnesLab-Connectors" package="1X07" value="" x="5" y="33" smashed="yes">
+<attribute name="NAME" x="3.73" y="34.397" size="0.6096" layer="25" font="vector" ratio="20"/>
+<attribute name="VALUE" x="3.73" y="30.968" size="0.6096" layer="27" font="vector" ratio="20"/>
 </element>
 </elements>
@@
 <wire x1="35.98" y1="5.08" x2="24.9682" y2="11.7348" width="0" layer="19" extent="1-1"/>
 <wire x1="4.0386" y1="31.9142" x2="20.27" y2="24.08" width="0" layer="19" extent="1-1"/>
-<wire x1="6.1976" y1="32.5882" x2="4.0386" y2="31.9142" width="0" layer="19" extent="1-1"/>
+<wire x1="7.1374" y1="14.986" x2="4.0386" y2="31.9142" width="0" layer="19" extent="1-1"/>
 </signal>
 <signal name="3.3V">
@@
 <wire x1="22.4282" y1="5.588" x2="21.1582" y2="5.588" width="0" layer="19" extent="1-1"/>
 <wire x1="4.0386" y1="30.2142" x2="4.7394" y2="23.5966" width="0" layer="19" extent="1-1"/>
-<wire x1="6.1976" y1="30.0482" x2="4.0386" y2="30.2142" width="0" layer="19" extent="1-1"/>
+<wire x1="7.1374" y1="12.446" x2="4.0386" y2="30.2142" width="0" layer="19" extent="1-1"/>
 <wire x1="37.68" y1="5.08" x2="22.4282" y2="5.588" width="0" layer="19" extent="1-1"/>
 </signal>
@@
 <contactref element="U1" pad="8"/>
 <contactref element="IMU1" pad="4"/>
-<wire x1="9.5446" y1="6.2818" x2="11.2776" y2="32.5882" width="0" layer="19" extent="1-1"/>
+<wire x1="9.5446" y1="6.2818" x2="12.2174" y2="14.986" width="0" layer="19" extent="1-1"/>
 <wire x1="24.9682" y1="5.588" x2="9.5446" y2="6.2818" width="0" layer="19" extent="1-1"/>
 </signal>
@@
 <contactref element="U1" pad="7"/>
 <contactref element="IMU1" pad="3"/>
-<wire x1="23.6982" y1="5.588" x2="11.2776" y2="30.0482" width="0" layer="19" extent="1-1"/>
+<wire x1="23.6982" y1="5.588" x2="12.2174" y2="12.446" width="0" layer="19" extent="1-1"/>
 <wire x1="9.5446" y1="3.929" x2="23.6982" y2="5.588" width="0" layer="19" extent="1-1"/>
 </signal>

Commit message: updated to 002
Connections:
- removed net LED.CTRL: U$4.8
- removed net PPG: C21.2, OP3.1, U1.14
- removed net TIA: C10.2, C15.1, OP4.1, U1.3
- new net A6/TIA: C10.2, C15.1, J1.5, OP4.1, U1.3
- new net A7/PPG: C21.2, J1.7, OP3.1, U1.14
- new net D29/LED.CTRL: J1.6, U$4.8
Changed lines of the file:
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@@
 <wire x1="9.5446" y1="3.929" x2="23.6982" y2="5.588" width="0" layer="19" extent="1-1"/>
 </signal>
-<signal name="TIA">
+<signal name="A6/TIA">
 <contactref element="C10" pad="2"/>
 <contactref element="U1" pad="3"/>
 <contactref element="C15" pad="1"/>
 <contactref element="OP4" pad="1"/>
+<contactref element="J1" pad="5"/>
 <wire x1="18.5166" y1="29.9584" x2="37.15" y2="24.094" width="0" layer="19" extent="1-1"/>
-<wire x1="13.3604" y1="29.3234" x2="18.5166" y2="29.9584" width="0" layer="19" extent="1-1"/>
+<wire x1="15.16" y1="33" x2="18.5166" y2="29.9584" width="0" layer="19" extent="1-1"/>
+<wire x1="13.3604" y1="29.3234" x2="15.16" y2="33" width="0" layer="19" extent="1-1"/>
 <wire x1="18.6182" y1="5.588" x2="13.3604" y2="29.3234" width="0" layer="19" extent="1-1"/>
 </signal>
@@
 <wire x1="2.7822" y1="4.1148" x2="7.5946" y2="3.929" width="0" layer="19" extent="1-1"/>
 </signal>
-<signal name="LED.CTRL">
+<signal name="D29/LED.CTRL">
 <contactref element="U$4" pad="8"/>
+<contactref element="J1" pad="6"/>
+<wire x1="7.5946" y1="6.2818" x2="17.7" y2="33" width="0" layer="19" extent="1-1"/>
 </signal>
 <signal name="N$10">
@@
 <contactref element="U1" pad="1"/>
 </signal>
-<signal name="PPG">
+<signal name="A7/PPG">
 <contactref element="U1" pad="14"/>
 <contactref element="C21" pad="2"/>
 <contactref element="OP3" pad="1"/>
-<wire x1="18.6182" y1="11.7348" x2="37.68" y2="10.16" width="0" layer="19" extent="1-1"/>
-<wire x1="14.9006" y1="26.3144" x2="18.6182" y2="11.7348" width="0" layer="19" extent="1-1"/>
+<contactref element="J1" pad="7"/>
+<wire x1="14.9006" y1="26.3144" x2="20.24" y2="33" width="0" layer="19" extent="1-1"/>
+<wire x1="18.6182" y1="11.7348" x2="14.9006" y2="26.3144" width="0" layer="19" extent="1-1"/>
+<wire x1="37.68" y1="10.16" x2="18.6182" y2="11.7348" width="0" layer="19" extent="1-1"/>
 </signal>
 <signal name="N$13">

Commit message: checkpoint 3
Parts:
- added C1: 100n, LinnesLab-Passives:C0603
- J1: device LinnesLab-Connectors:1X07 -> LinnesLab-Connectors:1X07_1.27MM
- moved R16 29.7 mm to (18.9, 29.5)
- moved C15 29.0 mm to (29.3, 4.27), turned to 0 degrees
- moved R13 27.9 mm to (32.9, 5.61), turned to 270 degrees
- moved C22 27.3 mm to (14.4, 20.6), turned to 90 degrees
- moved C14 22.1 mm to (29.3, 7.69), turned to 180 degrees
- moved OP4 21.9 mm to (16.8, 20.2)
- moved R19 21.9 mm to (32.9, 8.85), turned to 270 degrees
- moved R17 20.9 mm to (24.6, 19.4), turned to 90 degrees
- moved Q1 20.4 mm to (19.0, 27.0), turned to 180 degrees
- moved C20 20.4 mm to (21.6, 6.80), turned to 270 degrees
- moved R20 19.4 mm to (29.3, 5.95), turned to 180 degrees
- moved C11 19.4 mm to (25.1, 8.21), turned to 90 degrees
- moved R14 19.2 mm to (29.2, 9.31), turned to 0 degrees
- moved R18 19.2 mm to (23.3, 19.4), turned to 270 degrees
- moved C16 18.5 mm to (33.8, 13.9), turned to 90 degrees
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Connections:
- removed net LED: Q1.3
- net 3.3V: now also J1.4
- net A6/TIA: now also J1.6; no longer J1.5
- net D29/LED.CTRL: now also J1.5; no longer J1.6
- net GND: now also C1.1, J1.3
- net LED.C: now also Q1.3
- net SCL: now also J1.2
- net SDA: now also J1.1
- net VREF: now also C1.2
Routing:
- net A6/TIA: track 0.00 -> 56.2 mm, vias 0 -> 4
- net A7/PPG: track 0.00 -> 49.4 mm
- net VREF: track 0.00 -> 42.6 mm, vias 0 -> 2
- net SCL: track 0.00 -> 41.9 mm, vias 0 -> 6
- net SDA: track 0.00 -> 34.6 mm, vias 0 -> 2
- net PD.C: track 0.00 -> 26.7 mm, vias 0 -> 2
- net GND: track 0.00 -> 26.2 mm, vias 0 -> 15
- net N$19: track 0.00 -> 21.0 mm, vias 0 -> 2
- net N$9: track 0.00 -> 20.6 mm
- net G.W2: track 0.00 -> 17.4 mm, vias 0 -> 2
- net D29/LED.CTRL: track 0.00 -> 16.5 mm, vias 0 -> 2
- net N$13: track 0.00 -> 15.2 mm
- net 3.3V: track 0.00 -> 12.2 mm, vias 0 -> 2
- net N$17: track 0.00 -> 10.8 mm
- net N$16: track 0.00 -> 8.53 mm
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- added copper zone on layer 1, net 3.3V
- added copper zone on layer 16, net GND

Commit message: push onto repo
Parts:
- added C2, C5, C6: 1u, LinnesLab-Passives:C0603
- added C3, C4: 4.7u, LinnesLab-Passives:C0603
- added CHRG: MCP73831, LinnesLab-Power:SOT23-5
- added LDO2: MIC5504, LinnesLab-Power:SOT23-5
- added R1, R12: 100k, LinnesLab-Passives:R0603
- added R11: (no value), LinnesLab-Passives:R0603
- added U5: PCF8523, LinnesLab-Clocks:SO8
- added XTAL3: 32.7680kHz, LinnesLab-Clocks:2-SMD.NOLEAD.2.0MMTO1.2MM
Connections:
- new net D27/CHRGSTATUS: CHRG.1, R12.1
- new net N$1: U5.2, XTAL3.P$1
- new net N$2: U5.1, XTAL3.P$2
- new net N$3: CHRG.5, R11.2
- new net VBAT: U5.3
- new net VIN: C4.2, C5.2, CHRG.4, LDO2.1, LDO2.3, R12.2
- new net VLIPO: C3.1, CHRG.3
- net 3.3V: now also C2.1, C6.1, LDO2.5, R1.2, U5.8
- net GND: now also C2.2, C3.2, C4.1, C5.1, C6.2, CHRG.2, LDO2.2, R1.1, R11.1, U5.4
- net SCL: now also U5.6
- net SDA: now also U5.5

Commit message: Finished Top board with modifications
Parts:
- removed C3, C4: 4.7u, LinnesLab-Passives:C0603
- removed C5, C6: 1u, LinnesLab-Passives:C0603
- removed CHRG: MCP73831, LinnesLab-Power:SOT23-5
- removed LDO2: MIC5504, LinnesLab-Power:SOT23-5
- removed R1, R12: 100k, LinnesLab-Passives:R0603
- removed R11: (no value), LinnesLab-Passives:R0603
Connections:
- removed net D27/CHRGSTATUS: CHRG.1, R12.1
- removed net N$3: CHRG.5, R11.2
- removed net VIN: C4.2, C5.2, CHRG.4, LDO2.1, LDO2.3, R12.2
- removed net VLIPO: C3.1, CHRG.3
- net 3.3V: no longer C6.1, LDO2.5, R1.2
- net GND: no longer C3.2, C4.1, C5.1, C6.2, CHRG.2, LDO2.2, R1.1, R11.1
Changed lines of the file:
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@@
 <attribute name="VALUE" x="3.4798" y="-18.61311875" size="0.7112" layer="27"/>
-</element>
-<element name="CHRG" library="LinnesLab-Power" package="SOT23-5" value="MCP73831" x="4.815840625" y="-25.600659375" smashed="yes">
-<attribute name="NAME" x="2.910840625" y="-25.600659375" size="0.6096" layer="25" ratio="20" rot="R90" align="bottom-center"/>
-<attribute name="PROD_ID" value="IC-09995" x="4.815840625" y="-25.17901875" size="1.778" layer="27" display="off"/>
-<attribute name="VALUE" x="7.355840625" y="-25.600659375" size="0.6096" layer="27" ratio="20" rot="R90" align="bottom-center"/>
-</element>
-<element name="LDO2" library="LinnesLab-Power" package="SOT23-5" value="MIC5504" x="4.815840625" y="-38.13301875" smashed="yes">
-<attribute name="NAME" x="2.910840625" y="-38.13301875" size="0.6096" layer="25" ratio="20" rot="R90" align="bottom-center"/>
-<attribute name="VALUE" x="7.355840625" y="-38.13301875" size="0.6096" layer="27" ratio="20" rot="R90" align="bottom-center"/>
-</element>
-<element name="C5" library="LinnesLab-Passives" package="C0603" package3d_urn="urn:adsk.eagle:package:15661989/2" value="1u" x="3.5052" y="-33.733740625" smashed="yes">
-<attribute name="NAME" x="2.8702" y="-33.098740625" size="0.7112" layer="25"/>
-<attribute name="VALUE" x="2.8702" y="-35.638740625" size="0.7112" layer="27"/>
-</element>
-<element name="C6" library="LinnesLab-Passives" package="C0603" package3d_urn="urn:adsk.eagle:package:15661989/2" value="1u" x="6.5024" y="-33.733740625" smashed="yes">
-<attribute name="NAME" x="5.8674" y="-33.098740625" size="0.7112" layer="25"/>
-<attribute name="VALUE" x="5.8674" y="-35.638740625" size="0.7112" layer="27"/>
-</element>
-<element name="C3" library="LinnesLab-Passives" package="C0603" package3d_urn="urn:adsk.eagle:package:15661989/2" value="4.7u" x="6.80211875" y="-29.65958125" smashed="yes">
-<attribute name="NAME" x="6.16711875" y="-29.02458125" size="0.7112" layer="25"/>
-<attribute name="VALUE" x="6.16711875" y="-31.56458125" size="0.7112" layer="27"/>
-</element>
-<element name="C4" library="LinnesLab-Passives" package="C0603" package3d_urn="urn:adsk.eagle:package:15661989/2" value="4.7u" x="9.87551875" y="-29.65958125" smashed="yes">
-<attribute name="NAME" x="9.24051875" y="-29.02458125" size="0.7112" layer="25"/>
-<attribute name="VALUE" x="9.24051875" y="-31.56458125" size="0.7112" layer="27"/>
-</element>
-<element name="R11" library="LinnesLab-Passives" package="R0603" package3d_urn="urn:adsk.eagle:package:15661944/2" value="" x="9.362440625" y="-37.8079" smashed="yes">
-<attribute name="NAME" x="8.727440625" y="-37.1729" size="0.7112" layer="25"/>
-<attribute name="VALUE" x="8.727440625" y="-39.7129" size="0.7112" layer="27"/>
-</element>
-<element name="R12" library="LinnesLab-Passives" package="R0603" package3d_urn="urn:adsk.eagle:package:15661944/2" value="100k" x="9.362440625" y="-24.952959375" smashed="yes">
-<attribute name="NAME" x="8.727440625" y="-24.317959375" size="0.7112" layer="25"/>
-<attribute name="VALUE" x="8.727440625" y="-26.857959375" size="0.7112" layer="27"/>
-</element>
-<element name="R1" library="LinnesLab-Passives" package="R0603" package3d_urn="urn:adsk.eagle:package:15661944/2" value="100k" x="3.5052" y="-29.65958125" smashed="yes">
-<attribute name="NAME" x="2.8702" y="-29.02458125" size="0.7112" layer="25"/>
-<attribute name="VALUE" x="2.8702" y="-31.56458125" size="0.7112" layer="27"/>
 </element>
 </elements>
@@
 <contactref element="U5" pad="4"/>
 <contactref element="C2" pad="2"/>
-<contactref element="C5" pad="1"/>
-<contactref element="LDO2" pad="2"/>
-<contactref element="C6" pad="2"/>
-<contactref element="C3" pad="2"/>
-<contactref element="R11" pad="1"/>
-<contactref element="C4" pad="1"/>
-<contactref element="CHRG" pad="2"/>
-<contactref element="R1" pad="1"/>
 <wire x1="26.0604" y1="16.691921875" x2="32.222440625" y2="18.15248125" width="0" layer="19" extent="1-1"/>
 <wire x1="23.3019625" y1="20.012421875" x2="26.0604" y2="16.691921875" width="0" layer="19" extent="1-1"/>
@@
 <wire x1="2.7348" y1="-16.96211875" x2="10.795" y2="4.38911875" width="0" layer="19" extent="1-1"/>
 <wire x1="10.613759375" y1="-20.78228125" x2="2.7348" y2="-16.96211875" width="0" layer="19" extent="1-1"/>
-<wire x1="4.815840625" y1="-26.900759375" x2="10.613759375" y2="-20.78228125" width="0" layer="19" extent="1-1"/>
-<wire x1="2.6552" y1="-29.65958125" x2="4.815840625" y2="-26.900759375" width="0" layer="19" extent="1-1"/>
-<wire x1="7.65211875" y1="-29.65958125" x2="4.815840625" y2="-26.900759375" width="0" layer="19" extent="1-1"/>
-<wire x1="9.02551875" y1="-29.65958125" x2="7.65211875" y2="-29.65958125" width="0" layer="19" extent="1-1"/>
-<wire x1="2.6552" y1="-33.733740625" x2="2.6552" y2="-29.65958125" width="0" layer="19" extent="1-1"/>
-<wire x1="7.3524" y1="-33.733740625" x2="7.65211875" y2="-29.65958125" width="0" layer="19" extent="1-1"/>
-<wire x1="8.512440625" y1="-37.8079" x2="7.3524" y2="-33.733740625" width="0" layer="19" extent="1-1"/>
-<wire x1="4.815840625" y1="-39.43311875" x2="8.512440625" y2="-37.8079" width="0" layer="19" extent="1-1"/>
 </signal>
 <signal name="3.3V">
@@
 <contactref element="U5" pad="8"/>
 <contactref element="C2" pad="1"/>
-<contactref element="LDO2" pad="5"/>
-<contactref element="C6" pad="1"/>
-<contactref element="R1" pad="2"/>
 <wire x1="26.0604" y1="11.491921875" x2="32.219903125" y2="13.145403125" width="0" layer="19" extent="1-1"/>
 <wire x1="25.0672625" y1="9.056740625" x2="26.0604" y2="11.491921875" width="0" layer="19" extent="1-1"/>
@@
 <wire x1="8.0348" y1="-13.15211875" x2="6.46684375" y2="6.873240625" width="0" layer="19" extent="1-1"/>
 <wire x1="8.913759375" y1="-20.78228125" x2="8.0348" y2="-13.15211875" width="0" layer="19" extent="1-1"/>
-<wire x1="4.3552" y1="-29.65958125" x2="8.913759375" y2="-20.78228125" width="0" layer="19" extent="1-1"/>
-<wire x1="5.6524" y1="-33.733740625" x2="4.3552" y2="-29.65958125" width="0" layer="19" extent="1-1"/>
-<wire x1="3.865840625" y1="-36.83291875" x2="5.6524" y2="-33.733740625" width="0" layer="19" extent="1-1"/>
 </signal>
 <signal name="SDA">
@@
 <wire x1="2.7348" y1="-13.15211875" x2="5.14848125" y2="-20.99818125" width="0" layer="19" extent="1-1"/>
 </signal>
-<signal name="VIN">
-<contactref element="CHRG" pad="4"/>
-<contactref element="C5" pad="2"/>
-<contactref element="LDO2" pad="1"/>
-<contactref element="LDO2" pad="3"/>
-<contactref element="C4" pad="2"/>
-<contactref element="R12" pad="2"/>
-<wire x1="5.765840625" y1="-39.43311875" x2="3.865840625" y2="-39.43311875" width="0" layer="19" extent="1-1"/>
-<wire x1="4.3552" y1="-33.733740625" x2="3.865840625" y2="-39.43311875" width="0" layer="19" extent="1-1"/>
-<wire x1="10.72551875" y1="-29.65958125" x2="4.3552" y2="-33.733740625" width="0" layer="19" extent="1-1"/>
-<wire x1="10.212440625" y1="-24.952959375" x2="10.72551875" y2="-29.65958125" width="0" layer="19" extent="1-1"/>
-<wire x1="5.765840625" y1="-24.300559375" x2="10.212440625" y2="-24.952959375" width="0" layer="19" extent="1-1"/>
-</signal>
-<signal name="N$3">
-<contactref element="CHRG" pad="5"/>
-<contactref element="R11" pad="2"/>
-<wire x1="3.865840625" y1="-24.300559375" x2="10.212440625" y2="-37.8079" width="0" layer="19" extent="1-1"/>
-</signal>
-<signal name="VLIPO">
-<contactref element="CHRG" pad="3"/>
-<contactref element="C3" pad="1"/>
-<wire x1="5.765840625" y1="-26.900759375" x2="5.95211875" y2="-29.65958125" width="0" layer="19" extent="1-1"/>
-</signal>
-<signal name="D27/CHRGSTATUS">
-<contactref element="R12" pad="1"/>
-<contactref element="CHRG" pad="1"/>
-<wire x1="8.512440625" y1="-24.952959375" x2="3.865840625" y2="-26.900759375" width="0" layer="19" extent="1-1"/>
-</signal>
 </signals>

Commit message: finished bottom board
Parts:
- moved C2 58.5 mm to (32.0, 33.3), turned to 180 degrees
- moved XTAL3 55.6 mm to (25.7, 30.3), turned to 90 degrees
- moved U5 50.8 mm to (30.4, 29.2)
Connections:
- net A6/TIA renamed A5/TIA
- net A7/PPG renamed A4/PPG
- net D29/LED.CTRL renamed D30/LED.CTRL
Routing:
- net SDA: track 34.6 -> 66.6 mm, vias 2 -> 3
- net SCL: track 41.9 -> 71.1 mm, vias 6 -> 9
- net GND: track 26.2 -> 30.4 mm, vias 15 -> 17
- net N$1: track 0.00 -> 2.18 mm
- net N$2: track 0.00 -> 2.09 mm
