File: Hardware/Bottom/D2D-BOTTOM.sch (EAGLE design)
At the start: 31 parts, among them U1 AD5242-SO16

Commit message: unfinished 002
Parts:
- added J1: (no value), LinnesLab-Connectors:CONN_07
Other:
- moved on the sheet: C10, C11, C14, C15, C16, C17, C18, C19, C20, C21, C22, C24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

Commit message: updated to 002
Connections:
- removed net LED.CTRL: U$4.A
- removed net PPG: C21.2, OP3G$1.OUT, U1.B2
- removed net TIA: C10.2, C15.1, OP4G$1.OUT, U1.W1
- new net A6/TIA: C10.2, C15.1, J1.5, OP4G$1.OUT, U1.W1
- new net A7/PPG: C21.2, J1.7, OP3G$1.OUT, U1.B2
- new net D29/LED.CTRL: J1.6, U$4.A
Changed lines of the file:
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@@
 <setting verticaltext="up"/>
 </settings>
-<grid distance="1" unitdist="mil" unit="mm" style="lines" multiple="1" display="no" altdistance="0.01" altunitdist="inch" altunit="inch"/>
+<grid distance="0.1" unitdist="inch" unit="inch" style="lines" multiple="1" display="no" altdistance="0.01" altunitdist="inch" altunit="inch"/>
 <layers>
 <layer number="1" name="Top" color="4" fill="1" visible="no" active="no"/>
@@
 </segment>
 </net>
-<net name="TIA" class="0">
+<net name="A6/TIA" class="0">
 <segment>
 <wire x1="100.33" y1="25.146" x2="95.25" y2="25.146" width="0.1524" layer="91"/>
@@
 <junction x="47.625" y="98.8822"/>
 </segment>
+<segment>
+<pinref part="J1" gate="G$1" pin="5"/>
+<wire x1="86.36" y1="-12.7" x2="88.9" y2="-12.7" width="0.1524" layer="91"/>
+<label x="88.9" y="-12.7" size="1.27" layer="95" xref="yes"/>
+</segment>
 </net>
 <net name="PD.C" class="0">
@@
 </segment>
 </net>
-<net name="LED.CTRL" class="0">
+<net name="D29/LED.CTRL" class="0">
 <segment>
 <pinref part="U$4" gate="G$1" pin="A"/>
@@
 <wire x1="196.85" y1="27.686" x2="196.85" y2="35.306" width="0.1524" layer="91"/>
 <label x="196.85" y="35.306" size="1.27" layer="95" rot="R180" xref="yes"/>
+</segment>
+<segment>
+<pinref part="J1" gate="G$1" pin="6"/>
+<wire x1="86.36" y1="-10.16" x2="88.9254" y2="-10.16" width="0.1524" layer="91"/>
+<wire x1="88.9254" y1="-10.16" x2="88.9254" y2="-9.8806" width="0.1524" layer="91"/>
+<label x="88.9" y="-10.16" size="1.27" layer="95" xref="yes"/>
 </segment>
 </net>
@@
 </segment>
 </net>
-<net name="PPG" class="0">
+<net name="A7/PPG" class="0">
 <segment>
 <wire x1="128.27" y1="25.146" x2="130.81" y2="25.146" width="0.1524" layer="91"/>
@@
 <label x="187.325" y="91.2622" size="1.27" layer="95" xref="yes"/>
 </segment>
-</net>
+<segment>
+<pinref part="J1" gate="G$1" pin="7"/>
+<wire x1="86.36" y1="-7.62" x2="89.408" y2="-7.62" width="0.1524" layer="91"/>
+<wire x1="89.408" y1="-7.62" x2="89.408" y2="-7.5184" width="0.1524" layer="91"/>
+<label x="88.9" y="-7.62" size="1.27" layer="95" xref="yes"/>
+</segment>
+</net>

Commit message: checkpoint 3
Parts:
- added C1: 100n, LinnesLab-Passives:CAPACITOR0603
- J1: device LinnesLab-Connectors:CONN_07 -> LinnesLab-Connectors:CONN_07-1.27MM
Connections:
- removed net LED: Q1.C
- net 3.3V: now also J1.4
- net A6/TIA: now also J1.6; no longer J1.5
- net D29/LED.CTRL: now also J1.5; no longer J1.6
- net GND: now also C1.1, J1.3
- net LED.C: now also Q1.C
- net SCL: now also J1.2
- net SDA: now also J1.1
- net VREF: now also C1.2
Other:
- note added: "Castellated IMU breakout"
- note added: "Connection to digital potentiometer for dynamic gain control"
- note added: "Connection to optical sensor module"
- note added: "Connection to upper board"
- note added: "D2D PPG Circuit"
- note added: "Vref Generator and bypass capacitor"
- moved on the sheet: C24, IMU1, J1

Commit message: push onto repo
Parts:
- added C2, C5, C6: 1u, LinnesLab-Passives:CAPACITOR0603
- added C3, C4: 4.7u, LinnesLab-Passives:CAPACITOR0603
- added CHRG: MCP73831, LinnesLab-Power:MCP73831
- added LDO2: MIC5504, LinnesLab-Power:MIC5504
- added R1, R12: 100k, LinnesLab-Passives:RESISTOR0603
- added R11: (no value), LinnesLab-Passives:RESISTOR0603
- added U5: PCF8523, LinnesLab-Clocks:PCF8523
- added XTAL3: 32.7680kHz, LinnesLab-Clocks:CRYSTALECS-.327-12.5-12-C-TR
Connections:
- new net D27/CHRGSTATUS: CHRG.STAT, R12.1
- new net N$1: U5.OSCO, XTAL3.1
- new net N$2: U5.OSCI, XTAL3.2
- new net N$3: CHRG.PROG, R11.2
- new net VIN: C4.2, C5.2, CHRG.VIN, LDO2.EN, LDO2.IN, R12.2
- new net VLIPO: C3.1, CHRG.VBAT
- net 3.3V: now also C2.1, C6.1, LDO2.OUT, R1.2, U5.VDD
- net GND: now also C2.2, C3.2, C4.1, C5.1, C6.2, CHRG.VSS, LDO2.GND, R1.1, R11.1, U5.VSS
- net SCL: now also U5.SCL
- net SDA: now also U5.SDA
Other:
- note added: "Back-up battery if desired"
- note added: "I2C Address = 0x68h"
- note added: "Real-Time Clock"

Commit message: Finished Top board with modifications
Parts:
- removed C3, C4: 4.7u, LinnesLab-Passives:CAPACITOR0603
- removed C5, C6: 1u, LinnesLab-Passives:CAPACITOR0603
- removed CHRG: MCP73831, LinnesLab-Power:MCP73831
- removed LDO2: MIC5504, LinnesLab-Power:MIC5504
- removed R1, R12: 100k, LinnesLab-Passives:RESISTOR0603
- removed R11: (no value), LinnesLab-Passives:RESISTOR0603
Connections:
- removed net D27/CHRGSTATUS: CHRG.STAT, R12.1
- removed net N$3: CHRG.PROG, R11.2
- removed net VIN: C4.2, C5.2, CHRG.VIN, LDO2.EN, LDO2.IN, R12.2
- removed net VLIPO: C3.1, CHRG.VBAT
- net 3.3V: no longer C6.1, LDO2.OUT, R1.2
- net GND: no longer C3.2, C4.1, C5.1, C6.2, CHRG.VSS, LDO2.GND, R1.1, R11.1

Commit message: finished bottom board
Connections:
- net A6/TIA renamed A5/TIA
- net A7/PPG renamed A4/PPG
- net D29/LED.CTRL renamed D30/LED.CTRL
Changed lines of the file:
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@@
 </segment>
 </net>
-<net name="A6/TIA" class="0">
+<net name="A5/TIA" class="0">
 <segment>
 <wire x1="100.33" y1="25.146" x2="95.25" y2="25.146" width="0.1524" layer="91"/>
@@
 </segment>
 </net>
-<net name="D29/LED.CTRL" class="0">
+<net name="D30/LED.CTRL" class="0">
 <segment>
 <pinref part="U$4" gate="G$1" pin="A"/>
@@
 </segment>
 </net>
-<net name="A7/PPG" class="0">
+<net name="A4/PPG" class="0">
 <segment>
 <wire x1="128.27" y1="25.146" x2="130.81" y2="25.146" width="0.1524" layer="91"/>
